File: Schematics/ViBravo_September_2024/ViBravo_September_2024.kicad_pcb (KiCad board)
At the start: 2 copper layers, 65 x 70 mm, 44 parts, among them J1 Screw_Terminal_01x04, J3 Screw_Terminal_01x03, J4 Screw_Terminal_01x03, J5 Screw_Terminal_01x02, J6 Screw_Terminal_01x03, U1 LMV358IDR, U2 MAX7403CSA+, U3 LMV358IDR, U4 MAX7480ESA+

Commit message: pcb
Routing:
- net GND: track 330.1 -> 300.5 mm
- net USB: track 118.9 -> 118.2 mm

Commit message: updates to PCB
Parts:
- turned R8 to 0 degrees
Routing:
- net GND: track 300.5 -> 79.7 mm, vias 10 -> 9
- net A2: track 50.9 -> 106.8 mm, vias 2 -> 0
- net A1: track 39.3 -> 29.7 mm
- net BASS_OUT: track 25.8 -> 34.9 mm, vias 2 -> 0
- net Net-(U1-1OUT): track 22.1 -> 15.1 mm, vias 0 -> 2
- net Net-(U2-COM): track 11.3 -> 16.5 mm, vias 2 -> 0
- net 3V3: track 106.7 -> 102.5 mm
- net Net-(U2-CLK): track 11.9 -> 15.5 mm
- net A0: track 34.7 -> 31.7 mm, vias 2 -> 0
- net Net-(U4-COM): track 13.9 -> 16.6 mm, vias 2 -> 0
- net USB: track 118.2 -> 120.8 mm, vias 1 -> 3
- net Net-(U2-IN): track 57.2 -> 54.8 mm, vias 6 -> 2
- net Net-(J4-Pin_1): track 15.4 -> 13.4 mm
- net Net-(U2-OUT): track 9.06 -> 7.49 mm, vias 2 -> 0
- net Net-(U3-2IN-): track 22.2 -> 23.3 mm, vias 2 -> 0
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- added copper zone on B.Cu, net GND
Other:
- outline, holes or cut-outs redrawn

Commit message: updates to PCB
Parts:
- added REF**: MountingHole_2.5mm, MountingHole:MountingHole_2.5mm, F.Cu at (185.2, 63.8)
- added REF**: MountingHole_2.5mm, MountingHole:MountingHole_2.5mm, F.Cu at (185.2, 126.0)
- added REF**: MountingHole_2.5mm, MountingHole:MountingHole_2.5mm, F.Cu at (127.8, 63.8)
- added REF**: MountingHole_2.5mm, MountingHole:MountingHole_2.5mm, F.Cu at (127.8, 126.0)
Routing:
- net GND: track 79.7 -> 0.69 mm, vias 9 -> 19
- net A2: track 106.8 -> 50.4 mm, vias 0 -> 2
- net BASS_OUT: track 34.9 -> 22.8 mm, vias 0 -> 2
- net 3V3: track 102.5 -> 92.5 mm
- net USB: track 120.8 -> 115.4 mm
- net Net-(U2-IN): track 54.8 -> 53.4 mm, vias 2 -> 4
- net Net-(U2-COM): track 16.5 -> 15.2 mm
Other:
- outline, holes or cut-outs redrawn

Commit message: pcb updates
Parts:
- removed the REF** at (133.5, 70.7)
- removed the REF** at (153.8, 80.9)
- added J10: Screw_Terminal_01x04, TerminalBlock_TE-Connectivity:TerminalBlock_TE_282834-4_1x04_P2.54mm_Horizontal, F.Cu at (130.3, 101.1)
- added J6: Conn_01x16_Socket, Connector_PinSocket_2.54mm:PinSocket_1x16_P2.54mm_Vertical, F.Cu at (137.5, 70.7)
- added J7: Conn_01x12_Socket, Connector_PinSocket_2.54mm:PinSocket_1x12_P2.54mm_Vertical, F.Cu at (157.8, 80.9)
- added J8: Screw_Terminal_01x03, TerminalBlock_TE-Connectivity:TerminalBlock_TE_282834-3_1x03_P2.54mm_Horizontal, F.Cu at (182.6, 111.5)
- added R18: 10k, Resistor_SMD:R_1206_3216Metric, F.Cu at (180.1, 105.4)
- added R19: 10k, Resistor_SMD:R_1206_3216Metric, F.Cu at (184.9, 105.4)
- J1: renamed from J3; footprint TerminalBlock:TerminalBlock_bornier-3_P5.08mm -> TerminalBlock_TE-Connectivity:TerminalBlock_TE_282834-3_1x03_P2.54mm_Horizontal
- J2: renamed from J1; footprint TerminalBlock:TerminalBlock_bornier-4_P5.08mm -> TerminalBlock_TE-Connectivity:TerminalBlock_TE_282834-4_1x04_P2.54mm_Horizontal
- J3: renamed from J6; footprint TerminalBlock:TerminalBlock_bornier-3_P5.08mm -> TerminalBlock_TE-Connectivity:TerminalBlock_TE_282834-3_1x03_P2.54mm_Horizontal
- J4: footprint TerminalBlock:TerminalBlock_bornier-3_P5.08mm -> TerminalBlock_TE-Connectivity:TerminalBlock_TE_282834-3_1x03_P2.54mm_Horizontal
- J5: footprint TerminalBlock:TerminalBlock_bornier-2_P5.08mm -> TerminalBlock_TE-Connectivity:TerminalBlock_TE_282834-2_1x02_P2.54mm_Horizontal
- moved C11 23.6 mm to (179.8, 98.3)
- moved J4 13.1 mm to (164.7, 123.4), turned to 180 degrees
- moved R2 9.52 mm to (144.3, 115.3)
- moved J3 9.35 mm to (144.4, 123.4), turned to 180 degrees
- moved R17 7.93 mm to (169.8, 82.5)
- moved C15 5.94 mm to (175.3, 82.5)
- moved J5 5.70 mm to (173.9, 123.4), turned to 180 degrees
- moved C16 5.53 mm to (175.3, 78.2)
- moved R14 5.25 mm to (169.7, 78.3)
- moved R16 5.20 mm to (169.7, 74.4)
- moved C2 4.91 mm to (162.3, 82.8)
- moved R15 4.85 mm to (169.9, 86.4)
- moved J1 4.41 mm to (164.3, 66.8)
- moved C8 4.19 mm to (162.2, 86.4)
- moved R8 4.12 mm to (147.9, 86.1)
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- renumbered U3 to IC1, U2 to IC2, U1 to IC3, U4 to IC4
Routing:
- net SDA: track 0.00 -> 35.7 mm
- net SCL: track 0.00 -> 32.7 mm
- net BASS_OUT: track 22.8 -> 2.76 mm, vias 2 -> 0
- net Net-(J2-Pin_1): track 7.08 -> 24.5 mm
- net USB: track 115.4 -> 104.9 mm
- net Net-(IC1-1IN-): track 13.4 -> 22.8 mm
- net SCK: track 0.00 -> 9.24 mm
- net MO: track 0.00 -> 9.24 mm
- net MI: track 0.00 -> 9.24 mm
- net 3V3: track 92.5 -> 101.6 mm
- net A0: track 32.2 -> 29.3 mm
- net Net-(J3-Pin_3): track 9.15 -> 6.73 mm
- net Net-(C2-Pad2): track 8.94 -> 10.8 mm
- net A2: track 50.4 -> 48.7 mm
- net A1: track 29.8 -> 28.1 mm
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Other:
- board text added: "*"
- board text added: "Vibrosonics October 2024"

Commit message: updates to schematic
Parts:
- moved AUD_IN 30.7 mm to (115.3, 113.5), turned to 0 degrees
- moved VOL 30.5 mm to (135.9, 113.5), turned to 0 degrees
- moved LED 28.1 mm to (147.6, 113.5), turned to 0 degrees
- moved REF** 26.1 mm to (161.0, 116.0)
- moved REF** 26.1 mm to (161.0, 54.0)
- moved C9 25.8 mm to (155.3, 56.9)
- moved PWR 25.8 mm to (140.5, 56.9)
- moved C1 25.8 mm to (137.4, 108.1)
- moved C10 25.8 mm to (120.3, 100.1)
- moved C11 25.8 mm to (156.0, 88.4)
- moved C12 25.8 mm to (138.4, 84.1)
- moved C13 25.8 mm to (138.4, 88.1)
- moved C14 25.8 mm to (138.4, 80.6)
- moved C2 25.8 mm to (138.5, 72.9)
- moved C6 25.8 mm to (129.3, 81.1)
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- renumbered J3 to AUD_IN, J2 to AUD_OUT, J8 to I2C, J5 to LED, J1 to PWR, J10 to SPI, J4 to VOL
Connections:
- AUD_IN pad 1: Net-(J3-Pin_1) -> Net-(J3-Pin_3)
- AUD_IN pad 3: Net-(J3-Pin_3) -> Net-(J3-Pin_1)
- AUD_OUT pad 1: Net-(J2-Pin_1) -> GND
- AUD_OUT pad 2: Net-(J2-Pin_2) -> Net-(J2-Pin_3)
- AUD_OUT pad 3: Net-(J2-Pin_3) -> Net-(J2-Pin_2)
- AUD_OUT pad 4: GND -> Net-(J2-Pin_1)
- C9 pad 1: GND -> USB
- C9 pad 2: USB -> GND
- I2C pad 1: SCL -> GND
- I2C pad 3: GND -> SCL
- LED pad 1: Net-(J5-Pin_1) -> GND
- LED pad 2: GND -> Net-(J5-Pin_1)
- PWR pad 1: USB -> GND
- PWR pad 3: GND -> USB
- SPI pad 1: SCK -> GND
- SPI pad 2: MO -> SCK
- SPI pad 3: MI -> MO
- SPI pad 4: GND -> MI
- VOL pad 1: Net-(IC1-1IN-) -> GND
- VOL pad 3: GND -> Net-(IC1-1IN-)
Routing:
- net SCK: track 9.24 -> 10.5 mm
- net MI: track 9.24 -> 10.2 mm
- net MO: track 9.24 -> 10.2 mm
- net A2: track 48.7 -> 47.8 mm
- net Net-(IC1-1IN-): track 22.8 -> 23.4 mm
- net Net-(C2-Pad2): track 10.8 -> 10.2 mm
- net USB: track 104.9 -> 105.4 mm

Commit message: update to pcb and schematic
Parts:
- removed C9: 1000uF, Capacitor_THT:CP_Radial_D8.0mm_P3.50mm
- added C17: C_Polarized, Capacitor_THT:CP_Radial_D8.0mm_P3.50mm, F.Cu at (151.9, 56.9)
- turned R5 to 180 degrees
- turned R6 to 0 degrees
- renumbered PWR to J1, SPI to J10, AUD_OUT to J2, AUD_IN to J3, VOL to J4, LED to J5, I2C to J8
Connections:
- R5 pad 1: 3V3 -> Net-(IC3-1IN-)
- R5 pad 2: Net-(IC3-1IN-) -> GND
- R6 pad 1: Net-(IC3-1IN-) -> 3V3
- R6 pad 2: GND -> Net-(IC3-1IN-)
Routing:
- net USB: track 105.4 -> 100.7 mm
- net 3V3: track 101.2 -> 97.2 mm
- net Net-(IC3-1IN-): track 9.49 -> 10.0 mm
