File: Schematics/ViBravo_September_2024/ViBravo_September_2024.kicad_pcb (KiCad board)
At the start: 2 copper layers, 65 x 70 mm, 53 parts, among them IC1 LMV358IDR, IC2 MAX7403CSA+, IC3 LMV358IDR, IC4 MAX7480ESA+, J1 Screw_Terminal_01x03, J2 Screw_Terminal_01x04, J3 Screw_Terminal_01x03, J4 Screw_Terminal_01x03, J5 Screw_Terminal_01x02, J6 Conn_01x16_Socket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

Commit message: updates to PCB
Parts:
- added C18: 0.1uF, Capacitor_SMD:C_0805_2012Metric, F.Cu at (144.2, 108.1)
- R11: value 75 -> 150
- R5: value 47k -> 7.5k
- moved R19 36.1 mm to (125.1, 99.1), turned to 180 degrees
- moved R18 31.2 mm to (125.1, 96.3), turned to 180 degrees
- moved C11 11.8 mm to (147.7, 80.0), turned to 90 degrees
- moved C17 6.61 mm to (145.3, 56.9)
- moved J1 6.61 mm to (133.9, 56.9)
- moved R12 5.85 mm to (119.7, 94.6)
- moved R13 5.85 mm to (114.2, 94.6)
- moved C12 4.45 mm to (133.9, 84.3)
- moved C15 4.45 mm to (147.0, 72.6)
- moved C16 4.45 mm to (147.0, 68.3)
- moved IC3 4.45 mm to (145.0, 93.4)
- moved J4 4.45 mm to (131.5, 113.5)
- moved J5 4.45 mm to (143.2, 113.5)
- moved R15 4.45 mm to (141.6, 76.4)
- moved R16 4.45 mm to (141.4, 64.5)
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Connections:
- IC3 pad 8: 3V3 -> USB
- R11 pad 1: Net-(IC3-1OUT) -> Net-(J5-Pin_2)
- R11 pad 2: Net-(J5-Pin_2) -> Net-(IC3-1OUT)
- R18 pad 1: 3V3 -> SCL
- R18 pad 2: SCL -> 3V3
- R19 pad 1: 3V3 -> SDA
- R19 pad 2: SDA -> 3V3
- R6 pad 1: 3V3 -> USB
Routing:
- net 3V3: track 141.4 -> 88.3 mm, vias 4 -> 5
- net USB: track 100.7 -> 111.9 mm
- net SD_CS: track 58.4 -> 52.0 mm
- net BASS_OUT: track 2.76 -> 9.00 mm
- net Net-(J2-Pin_3): track 12.3 -> 17.0 mm
- net Net-(J2-Pin_2): track 13.4 -> 18.0 mm
- net Net-(IC4-COM): track 16.7 -> 13.8 mm, vias 0 -> 2
- net Net-(IC2-COM): track 14.6 -> 16.4 mm
- net SCL: track 32.7 -> 34.3 mm
- net Net-(IC3-1OUT): track 15.3 -> 13.7 mm
- net Net-(J5-Pin_2): track 9.31 -> 10.3 mm
- net SDA: track 35.7 -> 34.8 mm
- net GND: track 1.00 -> 0.10 mm, vias 25 -> 26
- net Net-(IC1-1IN+): track 16.1 -> 15.3 mm
Other:
- board text added: "Vibrosonics November 2024"
- board text removed: "Vibrosonics October 2024"

Commit message: updates to pcb
Parts:
- moved C17 2.29 mm to (147.6, 56.9)
- moved R18 1.27 mm to (125.2, 95.0)
- moved R12 0.46 mm to (119.6, 95.0)
- moved R13 0.46 mm to (114.1, 95.0)
- moved J1 0.38 mm to (134.3, 56.9)
- renumbered J2 to AUD_OUT
Routing:
- net USB: track 111.9 -> 113.6 mm
- net A2: track 47.8 -> 48.4 mm
- net SCL: track 34.3 -> 34.9 mm
Other:
- board text added: "+"
- board text added: "-"
- board text added: "- +"
- board text added: "3"
- board text added: "AUD_IN"
- board text added: "BASS"
- board text added: "I2C"
- board text added: "L R"
- board text added: "LED"
- board text added: "POT"
- board text added: "PWR"
- board text added: "SCL"
