File: Schematics/ViBravo_September_2024/ViBravo_September_2024.kicad_sch (KiCad schematic)
At the start: 45 parts, among them J1 Screw_Terminal_01x04, J3 Screw_Terminal_01x03, J4 Screw_Terminal_01x03, J5 Screw_Terminal_01x02, J6 Screw_Terminal_01x03, U1 LMV358IDR, U2 MAX7403CSA+, U3 LMV358IDR, U4 MAX7480ESA+

Commit message: pcb updates
Parts:
- removed A1: Adafruit_Feather_HUZZAH32_ESP32, Module:Adafruit_Feather, symbol MCU_Module:Adafruit_Feather_HUZZAH32_ESP32
- added J10: Screw_Terminal_01x04, TerminalBlock_TE-Connectivity:TerminalBlock_TE_282834-4_1x04_P2.54mm_Horizontal, symbol Connector:Screw_Terminal_01x04
- added J6: Conn_01x16_Socket, Connector_PinSocket_2.54mm:PinSocket_1x16_P2.54mm_Vertical, symbol Connector:Conn_01x16_Socket
- added J7: Conn_01x12_Socket, Connector_PinSocket_2.54mm:PinSocket_1x12_P2.54mm_Vertical, symbol Connector:Conn_01x12_Socket
- added J8, J9: Screw_Terminal_01x03, TerminalBlock_TE-Connectivity:TerminalBlock_TE_282834-3_1x03_P2.54mm_Horizontal, symbol Connector:Screw_Terminal_01x03
- added R18, R19: 10k, Resistor_SMD:R_1206_3216Metric, symbol Device:R
- J1: renamed from J3; footprint TerminalBlock:TerminalBlock_bornier-3_P5.08mm -> TerminalBlock_TE-Connectivity:TerminalBlock_TE_282834-3_1x03_P2.54mm_Horizontal
- J2: renamed from J1; footprint TerminalBlock:TerminalBlock_bornier-4_P5.08mm -> TerminalBlock_TE-Connectivity:TerminalBlock_TE_282834-4_1x04_P2.54mm_Horizontal
- J3: renamed from J6; footprint TerminalBlock:TerminalBlock_bornier-3_P5.08mm -> TerminalBlock_TE-Connectivity:TerminalBlock_TE_282834-3_1x03_P2.54mm_Horizontal
- J4: footprint TerminalBlock:TerminalBlock_bornier-3_P5.08mm -> TerminalBlock_TE-Connectivity:TerminalBlock_TE_282834-3_1x03_P2.54mm_Horizontal
- J5: footprint TerminalBlock:TerminalBlock_bornier-2_P5.08mm -> TerminalBlock_TE-Connectivity:TerminalBlock_TE_282834-2_1x02_P2.54mm_Horizontal
- renumbered U3 to IC1, U2 to IC2, U1 to IC3, U4 to IC4
Connections:
- net 3V3: now also J6.2 (Pin_2), R18.1, R19.1
- net A0: now also J6.5 (Pin_5)
- net A1: now also J6.6 (Pin_6)
- net A2: now also J6.7 (Pin_7)
- net GND: now also J10.4 (Pin_4), J6.4 (Pin_4), J8.3 (Pin_3), J9.3 (Pin_3)
- net USB: now also J7.3 (Pin_3)
- new net MI: J10.3 (Pin_3), J6.13 (Pin_13)
- new net MO: J10.2 (Pin_2), J6.12 (Pin_12)
- new net RX: J6.14 (Pin_14), J9.1 (Pin_1)
- new net SCK: J10.1 (Pin_1), J6.11 (Pin_11)
- new net SCL: J7.11 (Pin_11), J8.1 (Pin_1), R18.2
- new net SDA: J7.12 (Pin_12), J8.2 (Pin_2), R19.2
- new net TX: J6.15 (Pin_15), J9.2 (Pin_2)
Other:
- moved on the sheet: C12, C13, C14, C3, C4, C5, C6, C7, D1, IC2, IC3, IC4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

Commit message: updates to schematic
Parts:
- removed J9: Screw_Terminal_01x03, TerminalBlock_TE-Connectivity:TerminalBlock_TE_282834-3_1x03_P2.54mm_Horizontal, symbol Connector:Screw_Terminal_01x03
Connections:
- net GND: now also J1.1 (Pin_1), J10.1 (Pin_1), J2.1 (Pin_1), J4.1 (Pin_1), J5.1 (Pin_1), J8.1 (Pin_1); no longer J1.3 (Pin_3), J10.4 (Pin_4), J2.4 (Pin_4), J4.3 (Pin_3), J5.2 (Pin_2), J8.3 (Pin_3)
- net MI: now also J10.2 (Pin_2); no longer J10.3 (Pin_3)
- net MO: now also J10.3 (Pin_3); no longer J10.2 (Pin_2)
- net SCK: now also J10.4 (Pin_4); no longer J10.1 (Pin_1)
- net SCL: now also J8.3 (Pin_3); no longer J8.1 (Pin_1)
- net USB: now also J1.3 (Pin_3); no longer J1.1 (Pin_1)
- net at C11.2: now also J2.4 (Pin_4); no longer J2.1 (Pin_1)
- net at C16.2, R14.2: now also J2.3 (Pin_3); no longer J2.2 (Pin_2)
- net at C15.2, R15.2: now also J2.2 (Pin_2); no longer J2.3 (Pin_3)
- net at R11.2: now also J5.2 (Pin_2); no longer J5.1 (Pin_1)
- net at IC1.1 (1OUT), IC1.2 (1IN-): now also J4.3 (Pin_3); no longer J4.1 (Pin_1)
- net at R2.2: now also J3.3 (Pin_3); no longer J3.1 (Pin_1)
- net at R1.2: now also J3.1 (Pin_1); no longer J3.3 (Pin_3)
Other:
- moved on the sheet: J1, J2, J3, J4, J5

Commit message: update to pcb and schematic
Parts:
- removed C9: 1000uF, Capacitor_THT:CP_Radial_D8.0mm_P3.50mm, symbol Device:C
- added C17: C_Polarized, Capacitor_THT:CP_Radial_D8.0mm_P3.50mm, symbol Device:C_Polarized
Connections:
- net 3V3: now also R6.1; no longer R5.1
- net GND: now also R5.2, C17.2; no longer R6.2
- net MI: now also J10.4 (Pin_4); no longer J10.2 (Pin_2)
- net SCK: now also J10.2 (Pin_2); no longer J10.4 (Pin_4)
- net USB: now also C17.1
- new net: IC3.2 (1IN-), R5.1, R6.2
Other:
- moved on the sheet: R5, R6
Changed lines of the file:
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@@
 	)
 	(junction
-		(at 205.74 68.58)
+		(at 240.03 36.83)
 		(diameter 0)
 		(color 0 0 0 0)
 	)
 	(junction
-		(at 184.15 68.58)
+		(at 205.74 68.58)
 		(diameter 0)
 		(color 0 0 0 0)
 	)
 	(junction
-		(at 135.89 53.34)
+		(at 184.15 68.58)
 		(diameter 0)
 		(color 0 0 0 0)
 	)
 	(junction
-		(at 240.03 36.83)
+		(at 135.89 53.34)
 		(diameter 0)
 		(color 0 0 0 0)
@@
 	(wire
 		(pts
-			(xy 223.52 36.83) (xy 240.03 36.83)
-		)
-		(stroke
-			(width 0)
-			(type default)
-		)
-	)
-	(wire
-		(pts
 			(xy 43.18 132.08) (xy 43.18 134.62)
 		)
@@
 	(wire
 		(pts
+			(xy 223.52 36.83) (xy 240.03 36.83)
+		)
+		(stroke
+			(width 0)
+			(type default)
+		)
+	)
+	(wire
+		(pts
 			(xy 184.15 68.58) (xy 205.74 68.58)
 		)
@@
 	(global_label "MI"
 		(shape bidirectional)
-		(at 247.65 118.11 180)
+		(at 247.65 113.03 180)
 		(fields_autoplaced yes)
 		(effects
@@
 		)
 		(property "Intersheetrefs" "${INTERSHEET_REFS}"
-			(at 241.4973 118.11 0)
+			(at 241.4973 113.03 0)
 			(effects
 				(font
@@
 	(global_label "SCK"
 		(shape bidirectional)
-		(at 247.65 113.03 180)
+		(at 247.65 118.11 180)
 		(fields_autoplaced yes)
 		(effects
@@
 		)
 		(property "Intersheetrefs" "${INTERSHEET_REFS}"
-			(at 239.804 113.03 0)
+			(at 239.804 118.11 0)
 			(effects
 				(font
@@
 	(symbol
 		(lib_id "Device:R")
-		(at 240.03 40.64 0)
+		(at 240.03 33.02 0)
 		(unit 1)
 		(exclude_from_sim no)
@@
 		(fields_autoplaced yes)
 		(property "Reference" "R6"
-			(at 242.57 39.3699 0)
+			(at 242.57 31.7499 0)
 			(effects
 				(font
@@
 		)
 		(property "Value" "5k"
-			(at 242.57 41.9099 0)
+			(at 242.57 34.2899 0)
 			(effects
 				(font
@@
 		)
 		(property "Footprint" "Resistor_SMD:R_1206_3216Metric"
-			(at 238.252 40.64 90)
+			(at 238.252 33.02 90)
 			(effects
 				(font
@@
 		)
 		(property "Datasheet" "~"
-			(at 240.03 40.64 0)
+			(at 240.03 33.02 0)
 			(effects
 				(font
@@
 		)
 		(property "Description" "Resistor"
-			(at 240.03 40.64 0)
+			(at 240.03 33.02 0)
 			(effects
 				(font
@@
 	)
 	(symbol
+		(lib_id "Device:C_Polarized")
+		(at 54.61 129.54 0)
+		(unit 1)
+		(exclude_from_sim no)
+		(in_bom yes)
+		(on_board yes)
+		(dnp no)
+		(fields_autoplaced yes)
+		(property "Reference" "C17"
+			(at 58.42 127.3809 0)
+			(effects
+				(font
+					(size 1.27 1.27)
+				)
+				(justify left)
+			)
+		)
+		(property "Value" "C_Polarized"
+			(at 58.42 129.9209 0)
+			(effects
+				(font
+					(size 1.27 1.27)
+				)
+				(justify left)
+			)
+		)
+		(property "Footprint" "Capacitor_THT:CP_Radial_D8.0mm_P3.50mm"
+			(at 55.5752 133.35 0)
+			(effects
+				(font
+					(size 1.27 1.27)
+				)
+				(hide yes)
+			)
+		)
+		(property "Datasheet" "~"
+			(at 54.61 129.54 0)
+			(effects
+				(font
+					(size 1.27 1.27)
+				)
+				(hide yes)
+			)
+		)
+		(property "Description" "Polarized capacitor"
+			(at 54.61 129.54 0)
+			(effects
+				(font
+					(size 1.27 1.27)
+				)
+				(hide yes)
+			)
+		)
+		(pin "1"
+		)
+		(pin "2"
+		)
+		(instances
+			(project ""
+				(path "/c40baf00-5d70-4382-8f24-d28e6ebf545d"
+					(reference "C17")
+					(unit 1)
+				)
+			)
+		)
+	)
+	(symbol
 		(lib_id "power:GND")
 		(at 213.36 33.02 0)
@@
 	)
 	(symbol
-		(lib_id "Device:C")
-		(at 54.61 129.54 180)
-		(unit 1)
-		(exclude_from_sim no)
-		(in_bom yes)
-		(on_board yes)
-		(dnp no)
-		(fields_autoplaced yes)
-		(property "Reference" "C9"
-			(at 58.42 128.2699 0)
-			(effects
-				(font
-					(size 1.27 1.27)
-				)
-				(justify right)
-			)
-		)
-		(property "Value" "1000uF"
-			(at 58.42 130.8099 0)
-			(effects
-				(font
-					(size 1.27 1.27)
-				)
-				(justify right)
-			)
-		)
-		(property "Footprint" "Capacitor_THT:CP_Radial_D8.0mm_P3.50mm"
-			(at 53.6448 125.73 0)
-			(effects
-				(font
-					(size 1.27 1.27)
-				)
-				(hide yes)
-			)
-		)
-		(property "Datasheet" "~"
-			(at 54.61 129.54 0)
-			(effects
-				(font
-					(size 1.27 1.27)
-				)
-				(hide yes)
-			)
-		)
-		(property "Description" "Unpolarized capacitor"
-			(at 54.61 129.54 0)
-			(effects
-				(font
-					(size 1.27 1.27)
-				)
-				(hide yes)
-			)
-		)
-		(pin "2"
-		)
-		(pin "1"
-		)
-		(instances
-			(project "ViBravo_September_2024"
-				(path "/c40baf00-5d70-4382-8f24-d28e6ebf545d"
-					(reference "C9")
-					(unit 1)
-				)
-			)
-		)
-	)
-	(symbol
 		(lib_id "power:GND")
 		(at 54.61 134.62 0)
@@
 	(symbol
 		(lib_id "Device:R")
-		(at 240.03 33.02 0)
+		(at 240.03 40.64 0)
 		(unit 1)
 		(exclude_from_sim no)
@@
 		(fields_autoplaced yes)
 		(property "Reference" "R5"
-			(at 242.57 31.7499 0)
+			(at 242.57 39.3699 0)
 			(effects
 				(font
@@
 		)
 		(property "Value" "47k"
-			(at 242.57 34.2899 0)
+			(at 242.57 41.9099 0)
 			(effects
 				(font
@@
 		)
 		(property "Footprint" "Resistor_SMD:R_1206_3216Metric"
-			(at 238.252 33.02 90)
+			(at 238.252 40.64 90)
 			(effects
 				(font
@@
 		)
 		(property "Datasheet" "~"
-			(at 240.03 33.02 0)
+			(at 240.03 40.64 0)
 			(effects
 				(font
@@
 		)
 		(property "Description" "Resistor"
-			(at 240.03 33.02 0)
+			(at 240.03 40.64 0)
 			(effects
 				(font
