File: Schematics/ViBravo_September_2024/ViBravo_September_2024.kicad_sch (KiCad schematic)
At the start: 51 parts, among them IC1 LMV358IDR, IC2 MAX7403CSA+, IC3 LMV358IDR, IC4 MAX7480ESA+, J1 Screw_Terminal_01x03, J2 Screw_Terminal_01x04, J3 Screw_Terminal_01x03, J4 Screw_Terminal_01x03, J5 Screw_Terminal_01x02, J6 Conn_01x16_Socket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

Commit message: updates to PCB
Parts:
- R11: value 75 -> 150
- R5: value 47k -> 7.5k
Connections:
- net 3V3: now also R18.2, R19.2; no longer IC3.8 (VCC+), R18.1, R19.1, R6.1
- net SCL: now also R18.1; no longer R18.2
- net SDA: now also R19.1; no longer R19.2
- net USB: now also IC3.8 (VCC+), R6.1
- net at J5.2 (Pin_2): now also R11.1; no longer R11.2
- net at IC3.1 (1OUT): now also R11.2; no longer R11.1
Other:
- moved on the sheet: R11, R18, R19
