File: Schematics/AudioLux/AudioLux/AudioLux.kicad_sch (KiCad schematic)
At the start: 51 parts, among them IC1 LMV358IDR, IC2 MAX7403CSA+, IC3 LMV358IDR, IC4 MAX7480ESA+, J1 Screw_Terminal_01x03, J2 Screw_Terminal_01x04, J3 Screw_Terminal_01x03, J4 Screw_Terminal_01x03, J5 Screw_Terminal_01x02, J6 Conn_01x16_Socket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

Commit message: adding AudioLux
Parts:
- removed C11, C2, C8: 10uF, Capacitor_SMD:C_0805_2012Metric, symbol Device:C
- removed C12, C13, C15, C16: 0.1uF, Capacitor_SMD:C_0805_2012Metric, symbol Device:C
- removed C14: 6.8nF, Capacitor_SMD:C_0805_2012Metric, symbol Device:C
- removed IC4: MAX7480ESA+, 21-0041B_8_MXM, symbol 2024-10-15_04-05-58:MAX7480ESA+
- removed J2: Screw_Terminal_01x04, TerminalBlock_TE-Connectivity:TerminalBlock_TE_282834-4_1x04_P2.54mm_Horizontal, symbol Connector:Screw_Terminal_01x04
- removed J8: Screw_Terminal_01x03, TerminalBlock_TE-Connectivity:TerminalBlock_TE_282834-3_1x03_P2.54mm_Horizontal, symbol Connector:Screw_Terminal_01x03
- removed R14, R15: 3.3k, Resistor_SMD:R_1206_3216Metric, symbol Device:R
- removed R16, R17: 1.5k, Resistor_SMD:R_1206_3216Metric, symbol Device:R
Connections:
- net 3V3: now also R18.2, R19.2; no longer R18.1, R19.1
- net SCL: now also R18.1; no longer R18.2
- net SDA: now also R19.1; no longer R19.2
Other:
- moved on the sheet: R18, R19
